File: Hardware/calc-v2/calc-v2/calc-v2.kicad_pcb (KiCad board)
At the start: 2 copper layers, 82.6 x 128.3 mm, 74 parts, among them J1 ST-LINK, J2 LCD, SW1 0, SW10 -, SW11 4, SW12 5, SW13 6, SW14 *, SW15 /, SW16 7, SW17 8, SW18 9, SW19 EXP, SW2 /-/, SW20 C, SW21 sqrt, SW22 1/x, SW23 erf, SW24 R->P, SW25 Gamma(x), SW26 Cxy, SW27 y^x, SW28 ln, SW29 log, SW3 ., SW30 sin, SW31 cos, SW32 tan, SW33 Drop, SW34 X<>Y, SW35 DR, SW36 M+, SW37 MR, SW38 MS, SW39 F, SW4 +/-, SW40 G, SW41 Mode, SW42 Uncr, SW43 Prec, SW44 On, SW45 "Reset", SW5 ENTER, SW6 1, SW7 2, SW8 3, SW9 +, U1 TPS61222DCK, U2 STM32L476RETx, Y1 32.768 Hz

Commit message: Made all footprints handsolder-friendly
Parts:
- C1, C2: footprint SamacSys_Parts:CAPC1608X50N -> Capacitor_SMD:C_0603_1608Metric_Pad1.08x0.95mm_HandSolder
- C10, C12, C14: footprint SamacSys_Parts:CAPPC1709X100N -> Capacitor_SMD:C_0603_1608Metric_Pad1.08x0.95mm_HandSolder
- C11, C13, C3, C4, C5, C6, C8, C9: footprint SamacSys_Parts:CAPC1608X90N -> Capacitor_SMD:C_0603_1608Metric_Pad1.08x0.95mm_HandSolder
- C15, C7: footprint SamacSys_Parts:CAPC1608X87N -> Capacitor_SMD:C_0603_1608Metric_Pad1.08x0.95mm_HandSolder
- C16: footprint SamacSys_Parts:C0603 -> Capacitor_SMD:C_0603_1608Metric_Pad1.08x0.95mm_HandSolder
- D1, D2: footprint Diode_SMD:D_SOD-323 -> Diode_SMD:D_SOD-323_HandSoldering
- L1, L2, L3: footprint SamacSys_Parts:INDC2012X145N -> Inductor_SMD:L_0805_2012Metric_Pad1.15x1.40mm_HandSolder
- R2: footprint SamacSys_Parts:RESC1608X55N -> Capacitor_SMD:C_0603_1608Metric_Pad1.08x0.95mm_HandSolder
- moved R2 1.25 mm to (146.7, 60.7)
- moved C16 0.75 mm to (160.5, 35.2)
- moved C14 0.58 mm to (151.4, 69.9)
- moved C10 0.41 mm to (145.9, 57.2)
- moved C12 0.37 mm to (157.3, 51.9)
- moved C13 0.30 mm to (151.4, 68.4)

Commit message: Created 3D models for the EVQ switches
Parts:
- BT1: footprint foot-lib:BatteryHolder_Keystone_1057_1x2032 -> foot-lib:BatteryHolder_Keystone_1057
- moved L1 0.20 mm to (131.9, 55.7)
- moved U1 0.20 mm to (132.0, 51.9)
- moved C1 0.20 mm to (129.5, 51.9)
- moved C2 0.20 mm to (132.1, 49.5)
